Commit message: pizza transform

File: turtlebot3_simulations/turtlebot3_gazebo/urdf/HDL-32E.urdf.xacro (robot description, xacro)
@@ -1,6 +1,6 @@
 <?xml version="1.0"?>
-<robot xmlns:xacro="http://www.ros.org/wiki/xacro" name="VLP-16">
+<robot xmlns:xacro="http://www.ros.org/wiki/xacro" name="HDL-32E">
   <xacro:property name="M_PI" value="3.1415926535897931" />
-  <xacro:macro name="VLP-16" params="*origin parent:=base_link name:=velodyne tf_prefix:='' topic:=/velodyne_points organize_cloud:=false hz:=10 lasers:=16 samples:=1875 collision_range:=0.3 min_range:=0.9 max_range:=130.0 noise:=0.008 min_angle:=-${M_PI} max_angle:=${M_PI} gpu:=false">
+  <xacro:macro name="HDL-32E" params="*origin parent:=base_link name:=velodyne tf_prefix:='' topic:=/velodyne_points organize_cloud:=false hz:=10 lasers:=32 samples:=2187 collision_range:=0.3 min_range:=0.9 max_range:=130.0 noise:=0.008 min_angle:=-${M_PI} max_angle:=${M_PI} gpu:=false">
     <joint name="${name}_base_mount_joint" type="fixed">
       <xacro:insert_block name="origin" />
@@ -10,29 +10,24 @@
     <link name="${name}_base_link">
       <inertial>
-        <mass value="0.83"/>
-        <origin xyz="0 0 0.03585"/>
-        <inertia ixx="${(0.83 * (3.0*0.0516*0.0516 + 0.0717*0.0717)) / 12.0}" ixy="0" ixz="0"
-          iyy="${(0.83 * (3.0*0.0516*0.0516 + 0.0717*0.0717)) / 12.0}" iyz="0"
-          izz="${0.5 * 0.83 * (0.0516*0.0516)}"/>
+        <mass value="1.0"/>
+        <origin xyz="0 0 0.07212"/>
+        <inertia ixx="${(1.0 * (3.0*0.04267*0.04267 + 0.14424*0.14424)) / 12.0}" ixy="0" ixz="0"
+          iyy="${(1.0 * (3.0*0.04267*0.04267 + 0.14424*0.14424)) / 12.0}" iyz="0"
+          izz="${0.5 * 1.0 * (0.04267*0.04267)}"/>
       </inertial>
       <visual>
         <geometry>
-          <mesh filename="package://velodyne_description/meshes/VLP16_base_1.dae" />
-        </geometry>
-      </visual>
-      <visual>
-        <geometry>
-          <mesh filename="package://velodyne_description/meshes/VLP16_base_2.dae" />
+          <mesh filename="package://turtlebot3_gazebo/models/turtlebot3_waffle/meshes/HDL32E_base.dae" />
         </geometry>
       </visual>
       <collision>
-        <origin rpy="0 0 0" xyz="0 0 0.03585"/>
+        <origin rpy="0 0 0" xyz="0 0 0.07212"/>
         <geometry>
-          <cylinder radius="0.0516" length="0.0717"/>
+          <cylinder radius="0.04267" length="0.14424"/>
         </geometry>
       </collision>
     </link>
     <joint name="${name}_base_scan_joint" type="fixed" >
-      <origin xyz="0 0 0.0377" rpy="0 0 0" />
+      <origin xyz="0 0 0.09081" rpy="0 0 0" />
       <parent link="${name}_base_link" />
       <child link="${name}"/>
@@ -45,7 +40,7 @@
       </inertial>
       <visual>
-        <origin xyz="0 0 -0.0377" />
+        <origin xyz="0 0 -0.09081" rpy="0 0 0" />
         <geometry>
-          <mesh filename="package://velodyne_description/meshes/VLP16_scan.dae" />
+          <mesh filename="package://turtlebot3_gazebo/models/turtlebot3_waffle/meshes/HDL32E_scan.dae" />
         </geometry>
       </visual>
@@ -59,5 +54,5 @@
     <gazebo reference="${name}">
       <xacro:if value="${gpu}">
-        <sensor type="gpu_ray" name="${name}-VLP16">
+        <sensor type="gpu_ray" name="${name}-HDL32E">
           <pose>0 0 0 0 0 0</pose>
           <visualize>false</visualize>
@@ -74,6 +69,6 @@
                 <samples>${lasers}</samples>
                 <resolution>1</resolution>
-                <min_angle>-${15.0*M_PI/180.0}</min_angle>
-                <max_angle> ${15.0*M_PI/180.0}</max_angle>
+                <min_angle>-${30.67*M_PI/180.0}</min_angle>
+                <max_angle> ${10.67*M_PI/180.0}</max_angle>
               </vertical>
             </scan>
@@ -104,5 +99,5 @@
       </xacro:if>
       <xacro:unless value="${gpu}">
-        <sensor type="ray" name="${name}-VLP16">
+        <sensor type="ray" name="${name}-HDL32E">
           <pose>0 0 0 0 0 0</pose>
           <visualize>false</visualize>
@@ -119,6 +114,6 @@
                 <samples>${lasers}</samples>
                 <resolution>1</resolution>
-                <min_angle>-${15.0*M_PI/180.0}</min_angle>
-                <max_angle> ${15.0*M_PI/180.0}</max_angle>
+                <min_angle>-${30.67*M_PI/180.0}</min_angle>
+                <max_angle> ${10.67*M_PI/180.0}</max_angle>
               </vertical>
             </scan>

File: turtlebot3_simulations/turtlebot3_gazebo/urdf/VLP-16.urdf.xacro (robot description, xacro)
@@ -1,6 +1,6 @@
 <?xml version="1.0"?>
-<robot xmlns:xacro="http://www.ros.org/wiki/xacro" name="HDL-32E">
+<robot xmlns:xacro="http://www.ros.org/wiki/xacro" name="VLP-16">
   <xacro:property name="M_PI" value="3.1415926535897931" />
-  <xacro:macro name="HDL-32E" params="*origin parent:=base_link name:=velodyne tf_prefix:='' topic:=/velodyne_points organize_cloud:=false hz:=10 lasers:=32 samples:=2187 collision_range:=0.3 min_range:=0.9 max_range:=130.0 noise:=0.008 min_angle:=-${M_PI} max_angle:=${M_PI} gpu:=false">
+  <xacro:macro name="VLP-16" params="*origin parent:=base_link name:=velodyne tf_prefix:='' topic:=/velodyne_points organize_cloud:=false hz:=10 lasers:=16 samples:=1875 collision_range:=0.3 min_range:=0.9 max_range:=130.0 noise:=0.008 min_angle:=-${M_PI} max_angle:=${M_PI} gpu:=false">
     <joint name="${name}_base_mount_joint" type="fixed">
       <xacro:insert_block name="origin" />
@@ -10,24 +10,29 @@
     <link name="${name}_base_link">
       <inertial>
-        <mass value="1.0"/>
-        <origin xyz="0 0 0.07212"/>
-        <inertia ixx="${(1.0 * (3.0*0.04267*0.04267 + 0.14424*0.14424)) / 12.0}" ixy="0" ixz="0"
-          iyy="${(1.0 * (3.0*0.04267*0.04267 + 0.14424*0.14424)) / 12.0}" iyz="0"
-          izz="${0.5 * 1.0 * (0.04267*0.04267)}"/>
+        <mass value="0.83"/>
+        <origin xyz="0 0 0.03585"/>
+        <inertia ixx="${(0.83 * (3.0*0.0516*0.0516 + 0.0717*0.0717)) / 12.0}" ixy="0" ixz="0"
+          iyy="${(0.83 * (3.0*0.0516*0.0516 + 0.0717*0.0717)) / 12.0}" iyz="0"
+          izz="${0.5 * 0.83 * (0.0516*0.0516)}"/>
       </inertial>
       <visual>
         <geometry>
-          <mesh filename="package://velodyne_description/meshes/HDL32E_base.dae" />
+          <mesh filename="package://turtlebot3_gazebo/models/turtlebot3_waffle/meshes/VLP16_base_1.dae" />
+        </geometry>
+      </visual>
+      <visual>
+        <geometry>
+          <mesh filename="package://turtlebot3_gazebo/models/turtlebot3_waffle/meshes/VLP16_base_2.dae" />
         </geometry>
       </visual>
       <collision>
-        <origin rpy="0 0 0" xyz="0 0 0.07212"/>
+        <origin rpy="0 0 0" xyz="0 0 0.03585"/>
         <geometry>
-          <cylinder radius="0.04267" length="0.14424"/>
+          <cylinder radius="0.0516" length="0.0717"/>
         </geometry>
       </collision>
     </link>
     <joint name="${name}_base_scan_joint" type="fixed" >
-      <origin xyz="0 0 0.09081" rpy="0 0 0" />
+      <origin xyz="0 0 0.0377" rpy="0 0 0" />
       <parent link="${name}_base_link" />
       <child link="${name}"/>
@@ -40,7 +45,7 @@
       </inertial>
       <visual>
-        <origin xyz="0 0 -0.09081" rpy="0 0 0" />
+        <origin xyz="0 0 -0.0377" />
         <geometry>
-          <mesh filename="package://velodyne_description/meshes/HDL32E_scan.dae" />
+          <mesh filename="package://turtlebot3_gazebo/models/turtlebot3_waffle/meshes/VLP16_scan.dae" />
         </geometry>
       </visual>
@@ -54,5 +59,5 @@
     <gazebo reference="${name}">
       <xacro:if value="${gpu}">
-        <sensor type="gpu_ray" name="${name}-HDL32E">
+        <sensor type="gpu_ray" name="${name}-VLP16">
           <pose>0 0 0 0 0 0</pose>
           <visualize>false</visualize>
@@ -69,6 +74,6 @@
                 <samples>${lasers}</samples>
                 <resolution>1</resolution>
-                <min_angle>-${30.67*M_PI/180.0}</min_angle>
-                <max_angle> ${10.67*M_PI/180.0}</max_angle>
+                <min_angle>-${15.0*M_PI/180.0}</min_angle>
+                <max_angle> ${15.0*M_PI/180.0}</max_angle>
               </vertical>
             </scan>
@@ -99,5 +104,5 @@
       </xacro:if>
       <xacro:unless value="${gpu}">
-        <sensor type="ray" name="${name}-HDL32E">
+        <sensor type="ray" name="${name}-VLP16">
           <pose>0 0 0 0 0 0</pose>
           <visualize>false</visualize>
@@ -114,6 +119,6 @@
                 <samples>${lasers}</samples>
                 <resolution>1</resolution>
-                <min_angle>-${30.67*M_PI/180.0}</min_angle>
-                <max_angle> ${10.67*M_PI/180.0}</max_angle>
+                <min_angle>-${15.0*M_PI/180.0}</min_angle>
+                <max_angle> ${15.0*M_PI/180.0}</max_angle>
               </vertical>
             </scan>

File: turtlebot3_simulations/turtlebot3_gazebo/urdf/example.urdf.xacro (robot description, xacro)
@@ -32,9 +32,9 @@
     </inertial>
   </link>
-  <xacro:include filename="$(find velodyne_description)/urdf/VLP-16.urdf.xacro"/>
+  <xacro:include filename="$(find turtlebot3_gazebo)/urdf/VLP-16.urdf.xacro"/>
   <xacro:VLP-16 parent="base_link" name="velodyne" topic="/velodyne_points" organize_cloud="${organize_cloud}" hz="10" samples="440" gpu="${gpu}">
     <origin xyz="0 0 0.4" rpy="0 0 0" />
   </xacro:VLP-16>
-  <xacro:include filename="$(find velodyne_description)/urdf/HDL-32E.urdf.xacro"/>
+  <xacro:include filename="$(find turtlebot3_gazebo)/urdf/HDL-32E.urdf.xacro"/>
   <xacro:HDL-32E parent="base_link" name="velodyne2" topic="/velodyne_points2" organize_cloud="${organize_cloud}" hz="10" samples="220" gpu="${gpu}">
     <origin xyz="0 0 0.6" rpy="0 0 0" />
