Commit message: urdf -> urdf.xacro; velodyne added to urdf

File: turtlebot3_simulations/turtlebot3_gazebo/urdf/turtlebot3_waffle.urdf.xacro (robot description, xacro)
@@ -47,5 +47,5 @@
       <origin xyz="-0.064 0 0.0" rpy="0 0 0"/>
       <geometry>
-        <mesh filename="package://turtlebot3_gazebo/models/turtlebot3_waffle/meshes/waffle_base.stl" scale="0.001 0.001 0.001"/>
+        <mesh filename="package://turtlebot3_gazebo/models/turtlebot3_waffle/meshes/waffle_base.dae" scale="0.001 0.001 0.001"/>
       </geometry>
       <material name="light_black"/>
@@ -75,5 +75,5 @@
       <origin xyz="0 0 0" rpy="1.57 0 0"/>
       <geometry>
-        <mesh filename="package://turtlebot3_gazebo/models/turtlebot3_waffle/meshes/left_tire.stl" scale="0.001 0.001 0.001"/>
+        <mesh filename="package://turtlebot3_gazebo/models/turtlebot3_waffle/meshes/left_tire.dae" scale="0.001 0.001 0.001"/>
       </geometry>
       <material name="dark"/>
@@ -103,5 +103,5 @@
       <origin xyz="0 0 0" rpy="1.57 0 0"/>
       <geometry>
-        <mesh filename="package://turtlebot3_gazebo/models/turtlebot3_waffle/meshes/right_tire.stl" scale="0.001 0.001 0.001"/>
+        <mesh filename="package://turtlebot3_gazebo/models/turtlebot3_waffle/meshes/right_tire.dae" scale="0.001 0.001 0.001"/>
       </geometry>
       <material name="dark"/>
@@ -176,5 +176,5 @@
       <origin xyz="0 0 0" rpy="0 0 0"/>
       <geometry>
-        <mesh filename="package://turtlebot3_gazebo/models/turtlebot3_waffle/meshes/lds.stl" scale="0.001 0.001 0.001"/>
+        <mesh filename="package://turtlebot3_gazebo/models/turtlebot3_waffle/meshes/lds.dae" scale="0.001 0.001 0.001"/>
       </geometry>
       <material name="dark"/>
@@ -247,3 +247,16 @@
   </joint>
   <link name="camera_depth_optical_frame"/>
+  <!-- Velodyne part in xacro -->
+  <xacro:arg name="gpu" default="false"/>
+  <xacro:property name="gpu" value="$(arg gpu)" />
+  <xacro:arg name="organize_cloud" default="false"/>
+  <xacro:property name="organize_cloud" value="$(arg organize_cloud)" />
+  <xacro:include filename="$(find turtlebot3_gazebo)/urdf/VLP-16.urdf.xacro"/>
+  <xacro:VLP-16 parent="base_link" name="velodyne" topic="/velodyne_points" organize_cloud="${organize_cloud}" hz="10" samples="440" gpu="${gpu}">
+    <origin xyz="-0.064 0 0.2" rpy="0 0 0" />
+  </xacro:VLP-16>
+  <xacro:include filename="$(find turtlebot3_gazebo)/urdf/HDL-32E.urdf.xacro"/>
+  <xacro:HDL-32E parent="base_link" name="velodyne2" topic="/velodyne_points2" organize_cloud="${organize_cloud}" hz="10" samples="220" gpu="${gpu}">
+    <origin xyz="-0.064 0 0.3" rpy="0 0 0" />
+  </xacro:HDL-32E>
 </robot>
